Commit message: COMMIT Codice Semplificato MA NON PERFORMANTE

File: Evaluating/code/satellite.urdf (robot description, URDF)
Before this commit: robot satellite, 5 links, 4 joints
Links:
- link body: mass 500.0 -> 1000.0
- link left_arm: mass 10.0 -> 0.0
- link left_panel: mass 50.0 -> 0.0
- link right_arm: mass 10.0 -> 0.0
- link right_panel: mass 50.0 -> 0.0
